File: pcb/sensor_puck.kicad_sch (KiCad schematic)
At the start: 65 parts, among them J1 DISP LEFT, J2 DISP RIGHT, J3 USB_C_Receptacle_USB2.0_16P, J5 Generic, Q1 2N7002, SW1 RST, SW2 BOOT, U1 ESP32-S3-MINI-1U, U2 ST25DV16K-IER8C3, U3 LSM6DSOXTR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

Commit message: feat: PCB design v0.2
Parts:
- removed C11: 20uF, symbol Device:C
- removed F1, F2: Polyfuse, symbol Device:Polyfuse
- removed J5: Generic, Connector_PinHeader_2.54mm:PinHeader_1x04_P2.54mm_Vertical, symbol Connector:Conn_01x04_Socket
- removed TP3: 3V3, TestPoint:TestPoint_Pad_D1.0mm, symbol Connector:TestPoint
- removed TP4: GND, TestPoint:TestPoint_Pad_D1.0mm, symbol Connector:TestPoint
- removed TP9: VBUS, TestPoint:TestPoint_Pad_D1.0mm, symbol Connector:TestPoint
- added J6: Conn_01x02_Socket, Connector_PinHeader_2.00mm:PinHeader_1x02_P2.00mm_Vertical, symbol Connector:Conn_01x02_Socket
- added U4: SGP41-D-R4, SGP41-D-R4:XDCR_SGP41-D-R4, symbol SGP41-D-R4:SGP41-D-R4
- BZ1: footprint (none) -> Buzzer_Beeper:CMT-7525-80-SMT-TR
- C1, C12, C13, C19, C6, C8: JLCPCB Part # (none) -> C1711
- C10, C21: footprint (none) -> Capacitor_SMD:C_0805_2012Metric; JLCPCB Part # (none) -> C1710
- C17: footprint (none) -> Capacitor_SMD:C_0805_2012Metric; JLCPCB Part # (none) -> C5378
- C18, C20, C9: footprint (none) -> Capacitor_SMD:C_0805_2012Metric; JLCPCB Part # (none) -> C1711
- C2, C3: JLCPCB Part # (none) -> C28323
- C4, C5: value DNP -> 1uF; JLCPCB Part # (none) -> C28323
- C7: JLCPCB Part # (none) -> C1779
- D1: footprint (none) -> Diode_SMD:D_0805_2012Metric
- J3: JLCPCB Part # (none) -> C2988369
- L1: footprint (none) -> Connector_PinHeader_2.54mm:PinHeader_1x02_P2.54mm_Vertical
- Q1: JLCPCB Part # (none) -> C8545
- R1, R12, R2, R3, R7: JLCPCB Part # (none) -> C25612
- R10, R16, R17, R4: footprint (none) -> Resistor_SMD:R_0805_2012Metric; JLCPCB Part # (none) -> C25612
- R11: value TBD -> 5k11; footprint (none) -> Resistor_SMD:R_0805_2012Metric; JLCPCB Part # (none) -> C212414
- R15: value TBD -> 10k; footprint (none) -> Resistor_SMD:R_0805_2012Metric; JLCPCB Part # (none) -> C25612
- R5, R6: JLCPCB Part # (none) -> C212414
- R8: value 0 -> 10k; JLCPCB Part # (none) -> C25612
- R9: value 0 -> 4R7; JLCPCB Part # (none) -> C137423
- SW1, SW2: footprint Button_Switch_THT:SW_PUSH_6mm -> Button_Switch_SMD:SW_Push_1P1T_NO_CK_KMR2; JLCPCB Part # (none) -> C221676
- U3: footprint LSM6DSOX:PQFN50P250X300X86-14N -> Package_LGA:LGA-14_3x2.5mm_P0.5mm_LayoutBorder3x4y; Availability Not in stock -> In Stock; Description_1 Accelerometer, Gyroscope, 6 Axis Sensor I2C, SPI Output -> Accelerometer, Gyroscope, 6 Axis Sensor I2C, SPI Output
- U5: JLCPCB Part # (none) -> C47773
Connections:
- net +3V3: now also C5.1, D1.1 (K), J2.3 (Pin_3), R8.2, R9.2, U4.5 (VDDH)
- net BATT_READ: now also U1.14 (IO10); no longer U1.13 (IO9)
- net BUZZER_EN: now also U1.13 (IO9); no longer U1.15 (IO11)
- net GND: now also U4.2 (VSS), U4.4 (N/A), U4.7 (EXP)
- net I2C_SCL: now also J6.1 (Pin_1), U4.6 (SCL)
- net I2C_SDA: now also J6.2 (Pin_2), U4.3 (SDA)
- net LCD_CS: now also U1.33 (IO37); no longer U1.32 (IO36)
- net LCD_I2C_SCL: now also U1.11 (IO7); no longer R16.1, U1.9 (IO5)
- net LCD_I2C_SDA: now also R16.1, U1.12 (IO8); no longer U1.8 (IO4)
- net LIS2_INT: now also U1.10 (IO6); no longer U1.14 (IO10)
- net LSM6_INT1: now also U1.9 (IO5); no longer U1.12 (IO8)
- net LSM6_INT2: now also U1.8 (IO4); no longer U1.11 (IO7)
- net MISO: now also U1.16 (IO12); no longer U1.18 (IO14)
- net SD_CS: now also U1.32 (IO36); no longer U1.33 (IO37)
- net ST25DV_INT: now also R8.1, U1.15 (IO11)
- net TP_INT: now also U1.18 (IO14); no longer U1.16 (IO12)
- net USB_D+: now also J3.A6 (D+), J3.B6 (D+); no longer R9.1
- net USB_D-: now also J3.A7 (D-), J3.B7 (D-); no longer R8.2
- net VBUS: now also C3.2, C6.2, C7.2, J2.1 (Pin_1), J3.A4 (VBUS), J3.A9 (VBUS), J3.B4 (VBUS), J3.B9 (VBUS), U5.1 (VIN), U5.3 (EN); no longer D1.2 (A)
- net at BZ1.2 (-), Q1.3 (D): now also D1.2 (A)
- removed net VDC: C3.2, D1.1 (K), J2.1 (Pin_1), U5.1 (VIN), U5.3 (EN)
- new net: C4.1, R9.1, U4.1 (VDD)
- no-connect marks 18 -> 17
Other:
- note added: "CMT-7525-80-SMT-TR: 100mA max"
- note added: "I2C: 0x59"
- note added: "SGP41 - VOC / NOx Sensor"
- note added: "This transforms 5V to 3.309V, which _should_ be fine"
- note removed: "C11 from AliExpress devboard"
- note removed: "I_{hold} >= 500mA"
- note removed: "SMT-0825-S-HT-R: 80mA"
- note removed: "SeeedStudio ESP has 22R on D+/D- (?)"
- moved on the sheet: C10, C17, C18, C20, C21, C9, L1, R16, R17, R5, R6, U2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

Commit message: feat: update firmware for new PCB
Parts:
- U1: JLCPCB Part # (none) -> C22356044
- U3: JLCPCB Part # (none) -> C481766; MF STMicroelectronics -> (none); MP LSM6DSOXTR -> (none); PARTREV 3.0 -> (none); Package VFLGA-14 STMicroelectronics -> (none); Price None -> (none); Purchase-URL https://www.snapeda.com/api/url_track_click_mouser/?unipart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 -> (none); STANDARD IPC7351B -> (none); SnapEDA_Link https://www.snapeda.com/parts/LSM6DSOXTR/STMicroelectronics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 -> (none)
- U4: MAXIMUM_PACKAGE_HEIGHT 0.95 mm -> (none); MF Sensirion -> (none); MP SGP41-D-R4 -> (none); PARTREV 1.0 -> (none); Package None -> (none); Price None -> (none); STANDARD Manufacturer Recommendations -> (none); SnapEDA_Link https://www.snapeda.com/parts/SGP41-D-R4/Sensirion/view-par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 -> (none)
- U7: JLCPCB Part # (none) -> C919695
- U8: JLCPCB Part # (none) -> C3659294
Changed lines of the file:
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@@
 			)
 		)
-		(property "MF" "Sensirion"
-			(at 189.23 129.54 0)
-			(effects
-				(font
-					(size 1.27 1.27)
-				)
-				(justify bottom)
-				(hide yes)
-			)
-		)
-		(property "MAXIMUM_PACKAGE_HEIGHT" "0.95 mm"
-			(at 189.23 129.54 0)
-			(effects
-				(font
-					(size 1.27 1.27)
-				)
-				(justify bottom)
-				(hide yes)
-			)
-		)
-		(property "Package" "None"
-			(at 189.23 129.54 0)
-			(effects
-				(font
-					(size 1.27 1.27)
-				)
-				(justify bottom)
-				(hide yes)
-			)
-		)
-		(property "Price" "None"
-			(at 189.23 129.54 0)
-			(effects
-				(font
-					(size 1.27 1.27)
-				)
-				(justify bottom)
-				(hide yes)
-			)
-		)
 		(property "Check_prices" "https://www.snapeda.com/parts/SGP41-D-R4/Sensirion/view-part/?ref=eda"
 			(at 189.23 129.54 0)
@@
 			)
 		)
-		(property "STANDARD" "Manufacturer Recommendations"
-			(at 189.23 129.54 0)
-			(effects
-				(font
-					(size 1.27 1.27)
-				)
-				(justify bottom)
-				(hide yes)
-			)
-		)
-		(property "PARTREV" "1.0"
-			(at 189.23 129.54 0)
-			(effects
-				(font
-					(size 1.27 1.27)
-				)
-				(justify bottom)
-				(hide yes)
-			)
-		)
-		(property "SnapEDA_Link" "https://www.snapeda.com/parts/SGP41-D-R4/Sensirion/view-part/?ref=snap"
-			(at 189.23 129.54 0)
-			(effects
-				(font
-					(size 1.27 1.27)
-				)
-				(justify bottom)
-				(hide yes)
-			)
-		)
-		(property "MP" "SGP41-D-R4"
-			(at 189.23 129.54 0)
-			(effects
-				(font
-					(size 1.27 1.27)
-				)
-				(justify bottom)
-				(hide yes)
-			)
-		)
 		(property "Description_1" "\n                        \n                            Air Quality Sensor VOC and NOx Gas Sensor 3.3V 6-Pin DFN EP\n                        \n"
 			(at 189.23 129.54 0)
@@
 			)
 		)
-		(property "JLCPCB Part #" ""
+		(property "JLCPCB Part #" "C919695"
 			(at 252.73 124.46 0)
 			(effects
@@
 			)
 		)
-		(property "JLCPCB Part #" ""
+		(property "JLCPCB Part #" "C3659294"
 			(at 219.71 78.74 0)
 			(effects
@@
 			)
 		)
-		(property "JLCPCB Part #" ""
+		(property "JLCPCB Part #" "C22356044"
 			(at 99.06 66.04 0)
 			(effects
@@
 			)
 		)
-		(property "MF" "STMicroelectronics"
-			(at 226.06 41.91 0)
-			(effects
-				(font
-					(size 1.27 1.27)
-				)
-				(justify bottom)
-				(hide yes)
-			)
-		)
 		(property "Description_1" "\n                        \n                            Accelerometer, Gyroscope, 6 Axis Sensor I2C, SPI Output\n                        \n"
 			(at 226.06 41.91 0)
@@
 			)
 		)
-		(property "Package" "VFLGA-14 STMicroelectronics"
-			(at 226.06 41.91 0)
-			(effects
-				(font
-					(size 1.27 1.27)
-				)
-				(justify bottom)
-				(hide yes)
-			)
-		)
-		(property "Price" "None"
-			(at 226.06 41.91 0)
-			(effects
-				(font
-					(size 1.27 1.27)
-				)
-				(justify bottom)
-				(hide yes)
-			)
-		)
 		(property "Check_prices" "https://www.snapeda.com/parts/LSM6DSOXTR/STMicroelectronics/view-part/?ref=eda"
 			(at 226.06 41.91 0)
@@
 			)
 		)
-		(property "STANDARD" "IPC7351B"
-			(at 226.06 41.91 0)
-			(effects
-				(font
-					(size 1.27 1.27)
-				)
-				(justify bottom)
-				(hide yes)
-			)
-		)
-		(property "PARTREV" "3.0"
-			(at 226.06 41.91 0)
-			(effects
-				(font
-					(size 1.27 1.27)
-				)
-				(justify bottom)
-				(hide yes)
-			)
-		)
-		(property "SnapEDA_Link" "https://www.snapeda.com/parts/LSM6DSOXTR/STMicroelectronics/view-part/?ref=snap"
-			(at 226.06 41.91 0)
-			(effects
-				(font
-					(size 1.27 1.27)
-				)
-				(justify bottom)
-				(hide yes)
-			)
-		)
-		(property "MP" "LSM6DSOXTR"
-			(at 226.06 41.91 0)
-			(effects
-				(font
-					(size 1.27 1.27)
-				)
-				(justify bottom)
-				(hide yes)
-			)
-		)
-		(property "Purchase-URL" "https://www.snapeda.com/api/url_track_click_mouser/?unipart_id=3227828&manufacturer=STMicroelectronics&part_name=LSM6DSOXTR&search_term=None"
-			(at 226.06 41.91 0)
-			(effects
-				(font
-					(size 1.27 1.27)
-				)
-				(justify bottom)
-				(hide yes)
-			)
-		)
 		(property "Availability" "In Stock"
 			(at 226.06 41.91 0)
@@
 			)
 		)
-		(property "JLCPCB Part #" ""
+		(property "JLCPCB Part #" "C481766"
 			(at 226.06 41.91 0)
 			(effects
